File: SAMD21-breakout/SAMD21-breakout v1.sch (EAGLE design)
At the start: 8 parts, among them U1 ATSAMD21JTQFP

Commit message: New parts
Parts:
- U1: value ATSAMD21JTQFP -> AT-SAM-D21-JTQFP; device dr-library:ATSAMD21JTQFP -> dr-library:AT-SAM-D21-JTQFP
Connections:
- net GND: now also U1.GNDANA
Other:
- moved on the sheet: C1, L1
Changed lines of the file:
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@@
 </classes>
 <parts>
-<part name="U1" library="dr-library" deviceset="ATSAMD21J" device="TQFP"/>
 <part name="C1" library="dr-library" deviceset="CAP" device="0603" value="0.1uF"/>
 <part name="L1" library="dr-library" deviceset="INDUCTOR" device="0603"/>
@@
 <part name="GND2" library="supply1" deviceset="GND" device=""/>
 <part name="GND3" library="supply1" deviceset="GND" device=""/>
+<part name="U1" library="dr-library" deviceset="AT-SAM-D21-J" device="TQFP"/>
 </parts>
 <sheets>
@@
 </plain>
 <instances>
-<instance part="U1" gate="G$1" x="22.86" y="43.18"/>
-<instance part="C1" gate="G$1" x="-12.7" y="66.04"/>
-<instance part="L1" gate="G$1" x="-12.7" y="83.82" rot="R90"/>
+<instance part="C1" gate="G$1" x="-22.86" y="66.04"/>
+<instance part="L1" gate="G$1" x="-22.86" y="83.82" rot="R90"/>
 <instance part="R1" gate="G$1" x="-5.08" y="88.9" rot="R90"/>
 <instance part="C2" gate="G$1" x="30.48" y="111.76" rot="R90"/>
 <instance part="C3" gate="G$1" x="40.64" y="101.6" rot="R90"/>
 <instance part="C4" gate="G$1" x="45.72" y="96.52" rot="R90"/>
-<instance part="+3V1" gate="G$1" x="-12.7" y="99.06"/>
-<instance part="GND1" gate="1" x="-12.7" y="55.88"/>
+<instance part="+3V1" gate="G$1" x="-22.86" y="99.06"/>
+<instance part="GND1" gate="1" x="-22.86" y="55.88"/>
 <instance part="+3V2" gate="G$1" x="-5.08" y="101.6"/>
 <instance part="+3V3" gate="G$1" x="15.24" y="119.38"/>
@@
 <instance part="GND2" gate="1" x="55.88" y="91.44"/>
 <instance part="GND3" gate="1" x="25.4" y="-15.24"/>
+<instance part="U1" gate="G$1" x="22.86" y="43.18"/>
 </instances>
 <busses>
@@
 <net name="N$1" class="0">
 <segment>
+<wire x1="-2.54" y1="73.66" x2="-22.86" y2="73.66" width="0.1524" layer="91"/>
+<pinref part="L1" gate="G$1" pin="1"/>
+<wire x1="-22.86" y1="73.66" x2="-22.86" y2="76.2" width="0.1524" layer="91"/>
+<pinref part="C1" gate="G$1" pin="1"/>
+<wire x1="-22.86" y1="71.12" x2="-22.86" y2="73.66" width="0.1524" layer="91"/>
+<junction x="-22.86" y="73.66"/>
 <pinref part="U1" gate="G$1" pin="VDDANA"/>
-<wire x1="-2.54" y1="73.66" x2="-12.7" y2="73.66" width="0.1524" layer="91"/>
-<pinref part="L1" gate="G$1" pin="1"/>
-<wire x1="-12.7" y1="73.66" x2="-12.7" y2="76.2" width="0.1524" layer="91"/>
-<pinref part="C1" gate="G$1" pin="1"/>
-<wire x1="-12.7" y1="71.12" x2="-12.7" y2="73.66" width="0.1524" layer="91"/>
-<junction x="-12.7" y="73.66"/>
 </segment>
 </net>
 <net name="N$2" class="0">
 <segment>
-<pinref part="U1" gate="G$1" pin="RESET"/>
 <wire x1="-2.54" y1="78.74" x2="-5.08" y2="78.74" width="0.1524" layer="91"/>
 <pinref part="R1" gate="G$1" pin="1"/>
 <wire x1="-5.08" y1="78.74" x2="-5.08" y2="83.82" width="0.1524" layer="91"/>
+<pinref part="U1" gate="G$1" pin="RESET"/>
 </segment>
 </net>
@@
 <pinref part="+3V1" gate="G$1" pin="+3V3"/>
 <pinref part="L1" gate="G$1" pin="2"/>
-<wire x1="-12.7" y1="96.52" x2="-12.7" y2="91.44" width="0.1524" layer="91"/>
+<wire x1="-22.86" y1="96.52" x2="-22.86" y2="91.44" width="0.1524" layer="91"/>
 </segment>
 <segment>
 <pinref part="+3V3" gate="G$1" pin="+3V3"/>
-<pinref part="U1" gate="G$1" pin="VDDIN"/>
 <wire x1="15.24" y1="116.84" x2="15.24" y2="96.52" width="0.1524" layer="91"/>
-<pinref part="U1" gate="G$1" pin="VDDIO@48"/>
 <wire x1="15.24" y1="96.52" x2="15.24" y2="88.9" width="0.1524" layer="91"/>
 <wire x1="33.02" y1="88.9" x2="33.02" y2="96.52" width="0.1524" layer="91"/>
@@
 <junction x="33.02" y="96.52"/>
 <junction x="15.24" y="96.52"/>
-<pinref part="U1" gate="G$1" pin="VDDIO@34"/>
 <wire x1="30.48" y1="96.52" x2="27.94" y2="96.52" width="0.1524" layer="91"/>
 <wire x1="27.94" y1="96.52" x2="15.24" y2="96.52" width="0.1524" layer="91"/>
@@
 <wire x1="30.48" y1="101.6" x2="35.56" y2="101.6" width="0.1524" layer="91"/>
 <junction x="30.48" y="96.52"/>
-<pinref part="U1" gate="G$1" pin="VDDIO@21"/>
 <wire x1="27.94" y1="88.9" x2="27.94" y2="96.52" width="0.1524" layer="91"/>
 <pinref part="C5" gate="G$1" pin="1"/>
@@
 <wire x1="27.94" y1="106.68" x2="30.48" y2="106.68" width="0.1524" layer="91"/>
 <junction x="27.94" y="96.52"/>
+<pinref part="U1" gate="G$1" pin="VDDIO@48"/>
+<pinref part="U1" gate="G$1" pin="VDDIN"/>
+<pinref part="U1" gate="G$1" pin="VDDIO@34"/>
+<pinref part="U1" gate="G$1" pin="VDDIO@21"/>
 </segment>
 </net>
@@
 <pinref part="C1" gate="G$1" pin="2"/>
 <pinref part="GND1" gate="1" pin="GND"/>
-<wire x1="-12.7" y1="63.5" x2="-12.7" y2="58.42" width="0.1524" layer="91"/>
+<wire x1="-22.86" y1="63.5" x2="-22.86" y2="60.96" width="0.1524" layer="91"/>
+<pinref part="U1" gate="G$1" pin="GNDANA"/>
+<wire x1="-22.86" y1="60.96" x2="-22.86" y2="58.42" width="0.1524" layer="91"/>
+<wire x1="-2.54" y1="71.12" x2="-15.24" y2="71.12" width="0.1524" layer="91"/>
+<wire x1="-15.24" y1="71.12" x2="-15.24" y2="60.96" width="0.1524" layer="91"/>
+<wire x1="-15.24" y1="60.96" x2="-22.86" y2="60.96" width="0.1524" layer="91"/>
+<junction x="-22.86" y="60.96"/>
 </segment>
 <segment>
@@
 </segment>
 <segment>
-<pinref part="U1" gate="G$1" pin="GND@22"/>
 <wire x1="17.78" y1="-5.08" x2="17.78" y2="-7.62" width="0.1524" layer="91"/>
 <wire x1="17.78" y1="-7.62" x2="20.32" y2="-7.62" width="0.1524" layer="91"/>
@@
 <wire x1="22.86" y1="-7.62" x2="25.4" y2="-7.62" width="0.1524" layer="91"/>
 <wire x1="25.4" y1="-7.62" x2="25.4" y2="-12.7" width="0.1524" layer="91"/>
-<pinref part="U1" gate="G$1" pin="GND@47"/>
 <wire x1="22.86" y1="-5.08" x2="22.86" y2="-7.62" width="0.1524" layer="91"/>
 <junction x="22.86" y="-7.62"/>
-<pinref part="U1" gate="G$1" pin="GND@33"/>
 <wire x1="20.32" y1="-5.08" x2="20.32" y2="-7.62" width="0.1524" layer="91"/>
 <junction x="20.32" y="-7.62"/>
-<pinref part="U1" gate="G$1" pin="GND@54"/>
 <wire x1="25.4" y1="-5.08" x2="25.4" y2="-7.62" width="0.1524" layer="91"/>
 <junction x="25.4" y="-7.62"/>
+<pinref part="U1" gate="G$1" pin="GND@22"/>
+<pinref part="U1" gate="G$1" pin="GND@33"/>
+<pinref part="U1" gate="G$1" pin="GND@47"/>
+<pinref part="U1" gate="G$1" pin="GND@54"/>
 </segment>
 </net>
 <net name="N$7" class="0">
 <segment>
-<pinref part="U1" gate="G$1" pin="VDDCORE"/>
 <wire x1="17.78" y1="88.9" x2="17.78" y2="111.76" width="0.1524" layer="91"/>
 <pinref part="C2" gate="G$1" pin="1"/>
 <wire x1="25.4" y1="111.76" x2="17.78" y2="111.76" width="0.1524" layer="91"/>
+<pinref part="U1" gate="G$1" pin="VDDCORE"/>
 </segment>
 </net>
