File: ESP32 breakout/ESP32_breakout v1/ESP32_breakout v1.brd (EAGLE design)
At the start: 53.3 x 61 mm, 33 parts, among them U1 ESP-WROOM-32, Y1 12MHz

Commit message: Generate output files
Parts:
- U2: value (none) -> NCP-1117
Routing:
- net +3V3: track 135.1 -> 203.8 mm, vias 17 -> 18
- net IO4: track 47.1 -> 50.1 mm
- net IO5: track 30.0 -> 31.2 mm, vias 1 -> 0
- net IO2: track 52.3 -> 53.4 mm
- net IO15: track 46.5 -> 47.2 mm
- net VCC: vias 2 -> 3
- net RX: vias 4 -> 3
- net GND: vias 67 -> 69
Other:
- board text added: "3V3"
- board text added: "5V"
- board text added: "BOOT"
- board text added: "C6"
- board text added: "CLK"
- board text added: "CMD"
- board text added: "DRances"
- board text added: "EN"
- board text added: "ESP32 Breaakout v1"
- board text added: "GND"
- board text added: "IO0"
- board text added: "IO12"
- board text added: "IO13"
- board text added: "IO14"
- board text added: "IO15"
- board text added: "IO16"
- board text added: "IO17"
- board text added: "IO18"
- board text added: "IO19"
- board text added: "IO2"
- board text added: "IO21"
- board text added: "IO22"
- board text added: "IO23"
- board text added: "IO25"
- board text added: "IO26"
- board text added: "IO27"
- board text added: "IO34"
- board text added: "IO35"
- board text added: "IO4"
- board text added: "IO5"
- board text added: "May 15 2017"
- board text added: "RESET"
- board text added: "RX"
- board text added: "SD0"
- board text added: "SD1"
- board text added: "SD2"
- board text added: "SD3"
- board text added: "S_VN"
- board text added: "S_VP"
- board text added: "TX"
