File: ESP32 breakout/ESP32_breakout v1/ESP32_breakout v1.sch (EAGLE design)
At the start: 27 parts, among them U1 ESP-WROOM-32

Commit message: Generate output files
Parts:
- added U$14, U$15: M05, dr-library:M05
- U2: value (none) -> NCP-1117; device dr-library:REG-1117 -> dr-library:NCP-1117
- Y1: value (none) -> 12MHz
Connections:
- net CLK: now also U$14.1
- net CMD: now also U$15.5
- net GND: now also U$15.1
- net IO0: now also U$3.2; no longer U$3.1
- net IO13: now also U$15.2
- net IO15: now also U$14.4
- net IO16: now also U$3.4; no longer U$3.3
- net IO17: now also U$3.3; no longer U$3.4
- net IO18: now also U$3.5; no longer U$3.6
- net IO19: now also U$3.8; no longer U$3.7
- net IO2: now also U$14.5
- net IO21: now also U$3.7; no longer U$3.8
- net IO22: now also U$3.12; no longer U$3.11
- net IO23: now also U$3.11; no longer U$3.12
- net IO4: now also U$3.1; no longer U$3.2
- net IO5: now also U$3.6; no longer U$3.5
- net RX: now also U$3.10; no longer U$3.9
- net SD0: now also U$14.2
- net SD1: now also U$14.3
- net SD2: now also U$15.3
- net SD3: now also U$15.4
- net TX: now also U$3.9; no longer U$3.10
