File: SAML21 Breakout v1/SAML21 Breakout.brd (EAGLE design)
At the start: 100 x 80 mm, 23 parts, among them J1 M50-4910545, U1 AT-SAM-L21-JTQFP, Y2 32.768MHz

Commit message: Some changes
Parts:
- D1: value (none) -> PWR
Changed lines of the file:
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@@
 <element name="C8" library="dr-library" package="CAP-0603" value="10uF" x="51.435" y="14.605" rot="R90"/>
 <element name="C9" library="dr-library" package="CAP-0603" value="1uF" x="69.85" y="26.67"/>
-<element name="D1" library="dr-library" package="LED-1206" value="" x="50.8" y="40.64"/>
+<element name="D1" library="dr-library" package="LED-1206" value="PWR" x="50.8" y="40.64"/>
 <element name="J1" library="dr-library" package="M50-4910545" value="M50-4910545" x="69.85" y="41.91"/>
 <element name="L1" library="dr-library" package="IND-0603" value="" x="32.385" y="17.145"/>

Commit message: SAML21
Connections:
- new net 2.5V: U1.4
- net GND: now also J1.9
Changed lines of the file:
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@@
 <contactref element="J1" pad="3"/>
 <contactref element="J1" pad="5"/>
-<wire x1="69.85" y1="39.76" x2="68.6" y2="39.76" width="0" layer="19" extent="1-1"/>
+<contactref element="J1" pad="9"/>
+<wire x1="69.85" y1="39.76" x2="72.39" y2="39.76" width="0" layer="19" extent="1-1"/>
+<wire x1="68.6" y1="39.76" x2="69.85" y2="39.76" width="0" layer="19" extent="1-1"/>
 <wire x1="64.135" y1="33.274" x2="68.6" y2="39.76" width="0" layer="19" extent="1-1"/>
 <wire x1="59.69" y1="31.09" x2="64.135" y2="33.274" width="0" layer="19" extent="1-1"/>
@@
 <wire x1="70.739" y1="26.67" x2="64.38" y2="25.11" width="0" layer="19" extent="1-1"/>
 <wire x1="72.78" y1="22.86" x2="70.739" y2="26.67" width="0" layer="19" extent="1-1"/>
+<wire x1="52.55" y1="40.64" x2="55.245" y2="33.274" width="0" layer="19" extent="1-1"/>
 <wire x1="44.45" y1="30.099" x2="55.245" y2="33.274" width="0" layer="19" extent="1-1"/>
 <wire x1="42.545" y1="30.099" x2="44.45" y2="30.099" width="0" layer="19" extent="1-1"/>
@@
 <wire x1="33.02" y1="20.574" x2="36.16" y2="19.8" width="0" layer="19" extent="1-1"/>
 <wire x1="31.115" y1="20.574" x2="33.02" y2="20.574" width="0" layer="19" extent="1-1"/>
-<wire x1="52.55" y1="40.64" x2="55.245" y2="33.274" width="0" layer="19" extent="1-1"/>
 </signal>
 <signal name="N$3">
@@
 <wire x1="46.5075" y1="40.64" x2="49.05" y2="40.64" width="0" layer="19" extent="1-1"/>
 </signal>
+<signal name="2.5V">
+<contactref element="U1" pad="4"/>
+</signal>
 </signals>

Commit message: change
Parts:
- U2: value (none) -> AP7361C-33E-13
Changed lines of the file:
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@@
 <element name="S1" library="dr-library" package="SKHMQME010" value="" x="68.58" y="22.86"/>
 <element name="U1" library="dr-library" package="TQFP-64" value="AT-SAM-L21-JTQFP" x="41.91" y="19.05"/>
-<element name="U2" library="dr-library" package="SOT-223-3" value="" x="59.69" y="34.29"/>
+<element name="U2" library="dr-library" package="SOT-223-3" value="AP7361C-33E-13" x="59.69" y="34.29"/>
 <element name="Y2" library="dr-library" package="CFPX-217" value="32.768MHz" x="46.99" y="10.16" rot="R180"/>
 </elements>
