File: SAML21 Breakout v1/SAML21 Breakout.sch (EAGLE design)
At the start: 32 parts, among them J1 M50-4910545, U1 AT-SAM-L21-JTQFP, U2 AP7361C-33E-13, U3 MCP1501-CHY, Y2 32.768MHz

Commit message: Board layout started
Connections:
- removed net VREF: C15.1, C16.1, U$1.3
- net 2.5V: now also C15.1, C16.1, U$1.3
- net GND: no longer S1.3
Changed lines of the file:
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@@
 <pinref part="S1" gate="G$1" pin="1"/>
 <wire x1="-73.66" y1="53.34" x2="-73.66" y2="50.8" width="0.1524" layer="91"/>
-<pinref part="S1" gate="G$1" pin="3"/>
-<wire x1="-73.66" y1="58.42" x2="-71.12" y2="58.42" width="0.1524" layer="91"/>
-<wire x1="-71.12" y1="58.42" x2="-71.12" y2="50.8" width="0.1524" layer="91"/>
-<wire x1="-73.66" y1="50.8" x2="-71.12" y2="50.8" width="0.1524" layer="91"/>
-<wire x1="-71.12" y1="50.8" x2="-58.42" y2="50.8" width="0.1524" layer="91"/>
-<junction x="-71.12" y="50.8"/>
+<wire x1="-73.66" y1="50.8" x2="-58.42" y2="50.8" width="0.1524" layer="91"/>
 <pinref part="C9" gate="G$1" pin="2"/>
 <wire x1="-58.42" y1="50.8" x2="-58.42" y2="55.88" width="0.1524" layer="91"/>
@@
 </segment>
 </net>
-<net name="VREF" class="0">
+<net name="SHDN" class="0">
+<segment>
+<pinref part="VREF_EN" gate="G$1" pin="2"/>
+<wire x1="139.7" y1="12.7" x2="134.62" y2="12.7" width="0.1524" layer="91"/>
+<label x="134.62" y="12.7" size="1.778" layer="95"/>
+</segment>
+<segment>
+<pinref part="U3" gate="G$1" pin="SHDN"/>
+<wire x1="99.06" y1="12.7" x2="91.44" y2="12.7" width="0.1524" layer="91"/>
+<label x="91.44" y="12.7" size="1.778" layer="95"/>
+</segment>
+</net>
+<net name="N$7" class="0">
+<segment>
+<pinref part="VREF_EN" gate="G$1" pin="1"/>
+<wire x1="139.7" y1="10.16" x2="137.16" y2="10.16" width="0.1524" layer="91"/>
+<pinref part="R4" gate="G$1" pin="2"/>
+<wire x1="137.16" y1="10.16" x2="137.16" y2="7.62" width="0.1524" layer="91"/>
+</segment>
+</net>
+<net name="2.5V" class="0">
+<segment>
+<pinref part="U3" gate="G$1" pin="OUT"/>
+<wire x1="124.46" y1="15.24" x2="129.54" y2="15.24" width="0.1524" layer="91"/>
+<label x="124.46" y="15.24" size="1.778" layer="95"/>
+</segment>
 <segment>
 <pinref part="C16" gate="G$1" pin="1"/>
@@
 </segment>
 </net>
-<net name="SHDN" class="0">
-<segment>
-<pinref part="VREF_EN" gate="G$1" pin="2"/>
-<wire x1="139.7" y1="12.7" x2="134.62" y2="12.7" width="0.1524" layer="91"/>
-<label x="134.62" y="12.7" size="1.778" layer="95"/>
-</segment>
-<segment>
-<pinref part="U3" gate="G$1" pin="SHDN"/>
-<wire x1="99.06" y1="12.7" x2="91.44" y2="12.7" width="0.1524" layer="91"/>
-<label x="91.44" y="12.7" size="1.778" layer="95"/>
-</segment>
-</net>
-<net name="N$7" class="0">
-<segment>
-<pinref part="VREF_EN" gate="G$1" pin="1"/>
-<wire x1="139.7" y1="10.16" x2="137.16" y2="10.16" width="0.1524" layer="91"/>
-<pinref part="R4" gate="G$1" pin="2"/>
-<wire x1="137.16" y1="10.16" x2="137.16" y2="7.62" width="0.1524" layer="91"/>
-</segment>
-</net>
-<net name="2.5V" class="0">
-<segment>
-<pinref part="U3" gate="G$1" pin="OUT"/>
-<wire x1="124.46" y1="15.24" x2="129.54" y2="15.24" width="0.1524" layer="91"/>
-<label x="124.46" y="15.24" size="1.778" layer="95"/>
-</segment>
-</net>

Commit message: breakout
Parts:
- added JP1: M142ROWS, dr-library:M142ROWS
- added JP2, JP3, JP8: M122ROWS, dr-library:M122ROWS
- added JP4, JP5, JP6, JP7, JP9: M02LONG, dr-library:M02LONG
Connections:
- new net PA0: JP1.1, U1.PA00
- new net PA1: JP1.2, U1.PA01
- new net PA10: JP2.3, U1.PA10
- new net PA11: JP2.4, U1.PA11
- new net PA12: JP2.11, U1.PA12
- new net PA13: JP2.12, U1.PA13
- new net PA16: JP8.1, U1.PA16
- new net PA17: JP8.2, U1.PA17
- new net PA18: JP8.3, U1.PA18
- new net PA19: JP8.4, U1.PA19
- new net PA2: JP1.3, U1.PA02
- new net PA20: JP8.7, U1.PA20
- new net PA21: JP8.8, U1.PA21
- new net PA22: JP8.9, U1.PA22
- new net PA23: JP8.10, U1.PA23
- new net PA24: JP8.11, U1.PA24
- new net PA25: JP8.12, U1.PA25
- new net PA27: JP3.3, U1.PA27
- new net PA4: JP1.11, U1.PA04
- new net PA5: JP1.12, U1.PA05
- new net PA6: JP1.13, U1.PA06
- new net PA7: JP1.14, U1.PA07
- new net PA8: JP2.1, U1.PA08
- new net PA9: JP2.2, U1.PA09
- new net PB0: JP3.9, U1.PB00
- new net PB1: JP3.10, U1.PB01
- new net PB10: JP2.5, U1.PB10
- new net PB11: JP2.6, U1.PB11
- new net PB12: JP2.7, U1.PB12
- new net PB13: JP2.8, U1.PB13
- new net PB14: JP2.9, U1.PB14
- new net PB15: JP2.10, U1.PB15
- new net PB16: JP8.5, U1.PB16
- new net PB17: JP8.6, U1.PB17
- new net PB2: JP3.11, U1.PB02
- new net PB22: JP3.1, U1.PB22
- new net PB23: JP3.2, U1.PB23
- new net PB3: JP3.12, U1.PB03
- new net PB30: JP3.7, U1.PB30
- new net PB31: JP3.8, U1.PB31
- new net PB4: JP1.5, U1.PB04
- new net PB5: JP1.6, U1.PB05
- new net PB6: JP1.7, U1.PB06
- new net PB7: JP1.8, U1.PB07
- new net PB8: JP1.9, U1.PB08
- new net PB9: JP1.10, U1.PB09
- new net VSW: U1.VSW
- net +3V3: now also JP5.2, JP6.2, JP7.2, JP9.2
- net GND: now also JP4.2, JP5.1, JP6.1, JP7.1, JP9.1
- net RESET: now also JP3.4
- net SWCLK: now also JP3.5
- net SWDIO: now also JP3.6
- net VCC: now also JP4.1
- net VREF/PA3: now also JP1.4

Commit message: ddx
Parts:
- added D3, D4: PWR, dr-library:LED1206
- added JP10, JP11: M02, dr-library:M02
- added Q1, Q2: 2N7002, dr-library:2N7002
- added R6, R8: 330, dr-library:RESISTOR0603
- added R7, R9: 10k, dr-library:RESISTOR0603
Connections:
- new net HEART: JP10.2, Q1.D, R7.1
- new net HEART2: JP11.2, Q2.D, R9.1
- new net N$10: D4.A, R8.1
- new net N$11: D4.C, Q2.G
- new net N$8: D3.A, R6.1
- new net N$9: D3.C, Q1.G
- net +3V3: now also R6.2, R8.2
- net GND: now also Q1.S, Q2.S, R7.2, R9.2
- net PA8: now also JP10.1
- net PB10: now also JP11.1
Changed lines of the file:
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@@
 <part name="GND20" library="supply1" deviceset="GND" device=""/>
 <part name="+3V14" library="supply1" deviceset="+3V3" device=""/>
+<part name="Q1" library="dr-library" deviceset="2N7002" device=""/>
+<part name="R6" library="dr-library" deviceset="RESISTOR" device="0603" value="330"/>
+<part name="D3" library="dr-library" deviceset="LED" device="1206" value="PWR"/>
+<part name="+3V15" library="supply1" deviceset="+3V3" device=""/>
+<part name="GND21" library="supply1" deviceset="GND" device=""/>
+<part name="JP10" library="dr-library" deviceset="M02" device=""/>
+<part name="R7" library="dr-library" deviceset="RESISTOR" device="0603" value="10k"/>
+<part name="Q2" library="dr-library" deviceset="2N7002" device=""/>
+<part name="R8" library="dr-library" deviceset="RESISTOR" device="0603" value="330"/>
+<part name="D4" library="dr-library" deviceset="LED" device="1206" value="PWR"/>
+<part name="+3V16" library="supply1" deviceset="+3V3" device=""/>
+<part name="GND22" library="supply1" deviceset="GND" device=""/>
+<part name="JP11" library="dr-library" deviceset="M02" device=""/>
+<part name="R9" library="dr-library" deviceset="RESISTOR" device="0603" value="10k"/>
 </parts>
 <sheets>
@@
 <instance part="GND20" gate="1" x="167.64" y="88.9"/>
 <instance part="+3V14" gate="G$1" x="167.64" y="81.28"/>
+<instance part="Q1" gate="G$1" x="63.5" y="-73.66"/>
+<instance part="R6" gate="G$1" x="63.5" y="-48.26" rot="R90"/>
+<instance part="D3" gate="G$1" x="63.5" y="-58.42" rot="R270"/>
+<instance part="+3V15" gate="G$1" x="63.5" y="-38.1"/>
+<instance part="GND21" gate="1" x="63.5" y="-88.9"/>
+<instance part="JP10" gate="G$1" x="-35.56" y="-35.56"/>
+<instance part="R7" gate="G$1" x="58.42" y="-83.82"/>
+<instance part="Q2" gate="G$1" x="91.44" y="-73.66"/>
+<instance part="R8" gate="G$1" x="91.44" y="-48.26" rot="R90"/>
+<instance part="D4" gate="G$1" x="91.44" y="-58.42" rot="R270"/>
+<instance part="+3V16" gate="G$1" x="91.44" y="-38.1"/>
+<instance part="GND22" gate="1" x="91.44" y="-88.9"/>
+<instance part="JP11" gate="G$1" x="-7.62" y="-35.56"/>
+<instance part="R9" gate="G$1" x="86.36" y="-83.82"/>
 </instances>
 <busses>
@@
 <pinref part="GND19" gate="1" pin="GND"/>
 <wire x1="167.64" y1="73.66" x2="167.64" y2="71.12" width="0.1524" layer="91"/>
+</segment>
+<segment>
+<pinref part="Q1" gate="G$1" pin="S"/>
+<pinref part="GND21" gate="1" pin="GND"/>
+<wire x1="63.5" y1="-81.28" x2="63.5" y2="-83.82" width="0.1524" layer="91"/>
+<pinref part="R7" gate="G$1" pin="2"/>
+<wire x1="63.5" y1="-83.82" x2="63.5" y2="-86.36" width="0.1524" layer="91"/>
+<junction x="63.5" y="-83.82"/>
+</segment>
+<segment>
+<pinref part="Q2" gate="G$1" pin="S"/>
+<pinref part="GND22" gate="1" pin="GND"/>
+<wire x1="91.44" y1="-81.28" x2="91.44" y2="-83.82" width="0.1524" layer="91"/>
+<pinref part="R9" gate="G$1" pin="2"/>
+<wire x1="91.44" y1="-83.82" x2="91.44" y2="-86.36" width="0.1524" layer="91"/>
+<junction x="91.44" y="-83.82"/>
 </segment>
 </net>
@@
 <wire x1="167.64" y1="76.2" x2="167.64" y2="78.74" width="0.1524" layer="91"/>
 </segment>
+<segment>
+<pinref part="+3V15" gate="G$1" pin="+3V3"/>
+<pinref part="R6" gate="G$1" pin="2"/>
+<wire x1="63.5" y1="-40.64" x2="63.5" y2="-43.18" width="0.1524" layer="91"/>
+</segment>
+<segment>
+<pinref part="+3V16" gate="G$1" pin="+3V3"/>
+<pinref part="R8" gate="G$1" pin="2"/>
+<wire x1="91.44" y1="-40.64" x2="91.44" y2="-43.18" width="0.1524" layer="91"/>
+</segment>
 </net>
 <net name="N$1" class="0">
@@
 <pinref part="JP2" gate="G$1" pin="1"/>
 </segment>
+<segment>
+<pinref part="JP10" gate="G$1" pin="1"/>
+<wire x1="-30.48" y1="-33.02" x2="-20.32" y2="-33.02" width="0.1524" layer="91"/>
+<label x="-27.94" y="-33.02" size="1.778" layer="95"/>
+</segment>
 </net>
 <net name="PA9" class="0">
@@
 <label x="-55.88" y="-17.78" size="1.778" layer="95"/>
 </segment>
+<segment>
+<pinref part="JP11" gate="G$1" pin="1"/>
+<wire x1="-2.54" y1="-33.02" x2="7.62" y2="-33.02" width="0.1524" layer="91"/>
+<label x="0" y="-33.02" size="1.778" layer="95"/>
+</segment>
 </net>
 <net name="PB11" class="0">
@@
 </segment>
 </net>
+<net name="N$8" class="0">
+<segment>
+<pinref part="R6" gate="G$1" pin="1"/>
+<pinref part="D3" gate="G$1" pin="A"/>
+<wire x1="63.5" y1="-53.34" x2="63.5" y2="-55.88" width="0.1524" layer="91"/>
+</segment>
+</net>
+<net name="N$9" class="0">
+<segment>
+<pinref part="Q1" gate="G$1" pin="G"/>
+<pinref part="D3" gate="G$1" pin="C"/>
+<wire x1="63.5" y1="-66.04" x2="63.5" y2="-63.5" width="0.1524" layer="91"/>
+</segment>
+</net>
+<net name="HEART" class="0">
+<segment>
+<pinref part="Q1" gate="G$1" pin="D"/>
+<wire x1="55.88" y1="-76.2" x2="53.34" y2="-76.2" width="0.1524" layer="91"/>
+<label x="48.26" y="-76.2" size="1.778" layer="95"/>
+<pinref part="R7" gate="G$1" pin="1"/>
+<wire x1="53.34" y1="-76.2" x2="48.26" y2="-76.2" width="0.1524" layer="91"/>
+<wire x1="53.34" y1="-83.82" x2="53.34" y2="-76.2" width="0.1524" layer="91"/>
+<junction x="53.34" y="-76.2"/>
+</segment>
+<segment>
+<pinref part="JP10" gate="G$1" pin="2"/>
+<wire x1="-30.48" y1="-35.56" x2="-20.32" y2="-35.56" width="0.1524" layer="91"/>
+<label x="-27.94" y="-35.56" size="1.778" layer="95"/>
+</segment>
+</net>
+<net name="N$10" class="0">
+<segment>
+<pinref part="R8" gate="G$1" pin="1"/>
+<pinref part="D4" gate="G$1" pin="A"/>
+<wire x1="91.44" y1="-53.34" x2="91.44" y2="-55.88" width="0.1524" layer="91"/>
+</segment>
+</net>
+<net name="N$11" class="0">
+<segment>
+<pinref part="Q2" gate="G$1" pin="G"/>
+<pinref part="D4" gate="G$1" pin="C"/>
+<wire x1="91.44" y1="-66.04" x2="91.44" y2="-63.5" width="0.1524" layer="91"/>
+</segment>
+</net>
+<net name="HEART2" class="0">
+<segment>
+<pinref part="JP11" gate="G$1" pin="2"/>
+<wire x1="-2.54" y1="-35.56" x2="7.62" y2="-35.56" width="0.1524" layer="91"/>
+<label x="0" y="-35.56" size="1.778" layer="95"/>
+</segment>
+<segment>
+<pinref part="Q2" gate="G$1" pin="D"/>
+<wire x1="83.82" y1="-76.2" x2="81.28" y2="-76.2" width="0.1524" layer="91"/>
+<label x="76.2" y="-76.2" size="1.778" layer="95"/>
+<pinref part="R9" gate="G$1" pin="1"/>
+<wire x1="81.28" y1="-76.2" x2="76.2" y2="-76.2" width="0.1524" layer="91"/>
+<wire x1="81.28" y1="-83.82" x2="81.28" y2="-76.2" width="0.1524" layer="91"/>
+<junction x="81.28" y="-76.2"/>
+</segment>
+</net>

Commit message: component layout
Parts:
- added D5: VS-10BQ030-M3, dr-library:VS-10BQ030-M3
- added J2: (no value), EmbeddedAdventures 3:JACK-PLUG0
Connections:
- new net N$12: D5.A, J2.3
- net +3V3: no longer JP9.2
- net GND: now also J2.2, JP9.2; no longer JP9.1
- net VCC: now also D5.C, JP9.1
Other:
- moved on the sheet: JP9

Commit message: Added USB interface
Parts:
- added C17: 100nF, dr-library:CAP0603
- added R10, R11: 10k, dr-library:RESISTOR0603
- added U$6: MOLEX_USBMICRO, dr-library:MOLEX_USBMICRO
- added U4: TXS-0102-Q1, dr-library:TXS-0102-Q1
- added USB_EN: M03, dr-library:M03
Connections:
- removed net PA24: JP8.11, U1.PA24
- removed net PA25: JP8.12, U1.PA25
- new net N$13: R10.1, USB_EN.1
- new net N$14: U$6.D-, U4.B1
- new net N$15: U$6.D+, U4.B2
- new net N$17: R11.2, USB_EN.3
- new net N$19: U4.OE, USB_EN.2
- new net PA24/D-: JP8.11, U1.PA24, U4.A1
- new net PA25/D+: JP8.12, U1.PA25, U4.A2
- net +3V3: now also R10.2, U4.VA
- net GND: now also C17.2, R11.1, U$6.GND, U4.GND
- net VCC: now also C17.1, U$6.VDD, U4.VB
Other:
- note added: "Breakout Pins"
- note added: "External VREF"
- note added: "JTAG"
- note added: "LDO"
- note added: "Power Breakout"
- note added: "Programmable LED Reset button"
- note added: "SAML21J"
- note added: "USB Interface"
- moved on the sheet: C1, C10, C11, C12, C13, C14, C15, C16, C2, C3, C4, C5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

Commit message: pcb layout
Parts:
- removed U2: AP7361C-33E-13, dr-library:AP7361C-33E-13
- added U5: AP7362-33SP-13, dr-library:AP7362-33SP-13
- C12, C13: value 4.7uF -> 10uF
Connections:
- net +3V3: now also U5.OUT@5, U5.OUT@6, U5.OUT@7; no longer U2.VOUT
- net GND: now also U5.GND, U5.PAD; no longer U2.GND
- net PA3: now also JP1.4
- net VCC: now also U5.EN, U5.IN@3, U5.IN@4; no longer U2.VIN
- net VREF/PA3: no longer JP1.4
Other:
- moved on the sheet: C13, D1, R3
Changed lines of the file:
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@@
 <part name="Y2" library="dr-library" deviceset="LFXTAL054236-R" device="" value="32.768MHz"/>
 <part name="GND8" library="supply1" deviceset="GND" device=""/>
-<part name="U2" library="dr-library" deviceset="AP7361C-33E-13" device=""/>
-<part name="C12" library="dr-library" deviceset="CAP" device="0603" value="4.7uF"/>
-<part name="C13" library="dr-library" deviceset="CAP" device="0603" value="4.7uF"/>
+<part name="C12" library="dr-library" deviceset="CAP" device="0603" value="10uF"/>
+<part name="C13" library="dr-library" deviceset="CAP" device="0603" value="10uF"/>
 <part name="P+1" library="supply1" deviceset="VCC" device=""/>
 <part name="+3V6" library="supply1" deviceset="+3V3" device=""/>
@@
 <part name="R11" library="dr-library" deviceset="RESISTOR" device="0603" value="10k"/>
 <part name="GND25" library="supply1" deviceset="GND" device=""/>
+<part name="U5" library="dr-library" deviceset="AP7362-33SP-13" device=""/>
 </parts>
 <sheets>
@@
 <instance part="Y2" gate="G$1" x="187.96" y="71.12" rot="R90"/>
 <instance part="GND8" gate="1" x="170.18" y="66.04"/>
-<instance part="U2" gate="G$1" x="86.36" y="228.6"/>
 <instance part="C12" gate="G$1" x="71.12" y="220.98"/>
-<instance part="C13" gate="G$1" x="101.6" y="220.98"/>
+<instance part="C13" gate="G$1" x="106.68" y="220.98"/>
 <instance part="P+1" gate="VCC" x="71.12" y="238.76"/>
-<instance part="+3V6" gate="G$1" x="101.6" y="238.76"/>
-<instance part="GND9" gate="1" x="86.36" y="208.28"/>
-<instance part="R3" gate="G$1" x="114.3" y="228.6" rot="R90"/>
-<instance part="D1" gate="G$1" x="114.3" y="218.44" rot="R270"/>
-<instance part="GND10" gate="1" x="114.3" y="208.28"/>
+<instance part="+3V6" gate="G$1" x="106.68" y="238.76"/>
+<instance part="GND9" gate="1" x="88.9" y="208.28"/>
+<instance part="R3" gate="G$1" x="119.38" y="228.6" rot="R90"/>
+<instance part="D1" gate="G$1" x="119.38" y="218.44" rot="R270"/>
+<instance part="GND10" gate="1" x="119.38" y="208.28"/>
 <instance part="J1" gate="G$1" x="358.14" y="243.84"/>
 <instance part="+3V7" gate="G$1" x="337.82" y="256.54"/>
 <instance part="GND11" gate="1" x="337.82" y="231.14"/>
-<instance part="+3V8" gate="G$1" x="114.3" y="238.76"/>
+<instance part="+3V8" gate="G$1" x="119.38" y="238.76"/>
 <instance part="U3" gate="G$1" x="58.42" y="142.24"/>
 <instance part="C14" gate="G$1" x="40.64" y="139.7"/>
@@
 <instance part="R11" gate="G$1" x="309.88" y="167.64" rot="R90"/>
 <instance part="GND25" gate="1" x="309.88" y="157.48"/>
+<instance part="U5" gate="G$1" x="88.9" y="226.06"/>
 </instances>
 <busses>
@@
 </segment>
 <segment>
-<pinref part="C12" gate="G$1" pin="2"/>
-<wire x1="71.12" y1="218.44" x2="71.12" y2="215.9" width="0.1524" layer="91"/>
-<wire x1="71.12" y1="215.9" x2="86.36" y2="215.9" width="0.1524" layer="91"/>
-<pinref part="C13" gate="G$1" pin="2"/>
-<wire x1="86.36" y1="215.9" x2="101.6" y2="215.9" width="0.1524" layer="91"/>
-<wire x1="101.6" y1="215.9" x2="101.6" y2="218.44" width="0.1524" layer="91"/>
-<pinref part="U2" gate="G$1" pin="GND"/>
-<wire x1="86.36" y1="218.44" x2="86.36" y2="215.9" width="0.1524" layer="91"/>
-<junction x="86.36" y="215.9"/>
-<wire x1="86.36" y1="215.9" x2="86.36" y2="210.82" width="0.1524" layer="91"/>
-<pinref part="GND9" gate="1" pin="GND"/>
-</segment>
-<segment>
 <pinref part="GND10" gate="1" pin="GND"/>
 <pinref part="D1" gate="G$1" pin="C"/>
-<wire x1="114.3" y1="210.82" x2="114.3" y2="213.36" width="0.1524" layer="91"/>
+<wire x1="119.38" y1="210.82" x2="119.38" y2="213.36" width="0.1524" layer="91"/>
 </segment>
 <segment>
@@
 <wire x1="309.88" y1="162.56" x2="309.88" y2="160.02" width="0.1524" layer="91"/>
 <pinref part="GND25" gate="1" pin="GND"/>
+</segment>
+<segment>
+<pinref part="C12" gate="G$1" pin="2"/>
+<wire x1="71.12" y1="218.44" x2="71.12" y2="213.36" width="0.1524" layer="91"/>
+<wire x1="71.12" y1="213.36" x2="86.36" y2="213.36" width="0.1524" layer="91"/>
+<pinref part="GND9" gate="1" pin="GND"/>
+<wire x1="86.36" y1="213.36" x2="88.9" y2="213.36" width="0.1524" layer="91"/>
+<wire x1="88.9" y1="210.82" x2="88.9" y2="213.36" width="0.1524" layer="91"/>
+<pinref part="C13" gate="G$1" pin="2"/>
+<wire x1="106.68" y1="218.44" x2="106.68" y2="213.36" width="0.1524" layer="91"/>
+<wire x1="106.68" y1="213.36" x2="91.44" y2="213.36" width="0.1524" layer="91"/>
+<junction x="88.9" y="213.36"/>
+<pinref part="U5" gate="G$1" pin="GND"/>
+<wire x1="91.44" y1="213.36" x2="88.9" y2="213.36" width="0.1524" layer="91"/>
+<wire x1="86.36" y1="215.9" x2="86.36" y2="213.36" width="0.1524" layer="91"/>
+<junction x="86.36" y="213.36"/>
+<pinref part="U5" gate="G$1" pin="PAD"/>
+<wire x1="91.44" y1="215.9" x2="91.44" y2="213.36" width="0.1524" layer="91"/>
+<junction x="91.44" y="213.36"/>
 </segment>
 </net>
@@
 <pinref part="+3V6" gate="G$1" pin="+3V3"/>
 <pinref part="C13" gate="G$1" pin="1"/>
-<wire x1="101.6" y1="236.22" x2="101.6" y2="231.14" width="0.1524" layer="91"/>
-<pinref part="U2" gate="G$1" pin="VOUT"/>
-<wire x1="101.6" y1="231.14" x2="101.6" y2="226.06" width="0.1524" layer="91"/>
+<wire x1="106.68" y1="236.22" x2="106.68" y2="231.14" width="0.1524" layer="91"/>
+<wire x1="106.68" y1="231.14" x2="106.68" y2="226.06" width="0.1524" layer="91"/>
+<junction x="106.68" y="231.14"/>
+<pinref part="U5" gate="G$1" pin="OUT@5"/>
 <wire x1="99.06" y1="231.14" x2="101.6" y2="231.14" width="0.1524" layer="91"/>
+<pinref part="U5" gate="G$1" pin="OUT@7"/>
+<wire x1="101.6" y1="231.14" x2="106.68" y2="231.14" width="0.1524" layer="91"/>
+<wire x1="99.06" y1="226.06" x2="101.6" y2="226.06" width="0.1524" layer="91"/>
+<wire x1="101.6" y1="226.06" x2="101.6" y2="228.6" width="0.1524" layer="91"/>
 <junction x="101.6" y="231.14"/>
+<pinref part="U5" gate="G$1" pin="OUT@6"/>
+<wire x1="101.6" y1="228.6" x2="101.6" y2="231.14" width="0.1524" layer="91"/>
+<wire x1="99.06" y1="228.6" x2="101.6" y2="228.6" width="0.1524" layer="91"/>
+<junction x="101.6" y="228.6"/>
 </segment>
 <segment>
@@
 <segment>
 <pinref part="R3" gate="G$1" pin="2"/>
-<wire x1="114.3" y1="233.68" x2="114.3" y2="236.22" width="0.1524" layer="91"/>
+<wire x1="119.38" y1="233.68" x2="119.38" y2="236.22" width="0.1524" layer="91"/>
 <pinref part="+3V8" gate="G$1" pin="+3V3"/>
 </segment>
@@
 <pinref part="C12" gate="G$1" pin="1"/>
 <wire x1="71.12" y1="236.22" x2="71.12" y2="231.14" width="0.1524" layer="91"/>
-<pinref part="U2" gate="G$1" pin="VIN"/>
 <wire x1="71.12" y1="231.14" x2="71.12" y2="226.06" width="0.1524" layer="91"/>
-<wire x1="73.66" y1="231.14" x2="71.12" y2="231.14" width="0.1524" layer="91"/>
 <junction x="71.12" y="231.14"/>
 <pinref part="D5" gate="G$1" pin="C"/>
 <wire x1="68.58" y1="231.14" x2="71.12" y2="231.14" width="0.1524" layer="91"/>
+<pinref part="U5" gate="G$1" pin="IN@3"/>
+<wire x1="71.12" y1="231.14" x2="76.2" y2="231.14" width="0.1524" layer="91"/>
+<pinref part="U5" gate="G$1" pin="IN@4"/>
+<wire x1="76.2" y1="231.14" x2="78.74" y2="231.14" width="0.1524" layer="91"/>
+<wire x1="78.74" y1="228.6" x2="76.2" y2="228.6" width="0.1524" layer="91"/>
+<wire x1="76.2" y1="228.6" x2="76.2" y2="231.14" width="0.1524" layer="91"/>
+<junction x="76.2" y="231.14"/>
+<pinref part="U5" gate="G$1" pin="EN"/>
+<wire x1="78.74" y1="226.06" x2="76.2" y2="226.06" width="0.1524" layer="91"/>
+<wire x1="76.2" y1="226.06" x2="76.2" y2="228.6" width="0.1524" layer="91"/>
+<junction x="76.2" y="228.6"/>
 </segment>
 <segment>
@@
 <pinref part="D1" gate="G$1" pin="A"/>
 <pinref part="R3" gate="G$1" pin="1"/>
-<wire x1="114.3" y1="220.98" x2="114.3" y2="223.52" width="0.1524" layer="91"/>
+<wire x1="119.38" y1="220.98" x2="119.38" y2="223.52" width="0.1524" layer="91"/>
 </segment>
 </net>
@@
 <label x="88.9" y="124.46" size="1.778" layer="95"/>
 </segment>
+<segment>
+<wire x1="342.9" y1="116.84" x2="350.52" y2="116.84" width="0.1524" layer="91"/>
+<label x="345.44" y="116.84" size="1.778" layer="95"/>
+<pinref part="JP1" gate="G$1" pin="4"/>
+</segment>
 </net>
 <net name="VREF/PA3" class="0">
@@
 <label x="88.9" y="127" size="1.778" layer="95"/>
 </segment>
-<segment>
-<wire x1="342.9" y1="116.84" x2="350.52" y2="116.84" width="0.1524" layer="91"/>
-<label x="345.44" y="116.84" size="1.778" layer="95"/>
-<pinref part="JP1" gate="G$1" pin="4"/>
-</segment>
-</net>
+</net>
