File: SAML21 Breakout v1/SAML21 Breakout.sch (EAGLE design)
At the start: 59 parts, among them J1 M50-4910545, Q1 2N7002, Q2 2N7002, U1 AT-SAM-L21-JTQFP, U3 MCP1501-CHY, U4 TXS-0102-Q1, U5 AP7362-33SP-13, Y2 32.768MHz

Commit message: Component size change
Parts:
- R1, R10, R11, R2, R3, R4, R5, R6, R7, R8, R9: device dr-library:RESISTOR0603 -> dr-library:RESISTOR0805
Changed lines of the file:
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@@
 <part name="+3V5" library="supply1" deviceset="+3V3" device=""/>
 <part name="GND6" library="supply1" deviceset="GND" device=""/>
-<part name="R1" library="dr-library" deviceset="RESISTOR" device="0603" value="10k"/>
-<part name="R2" library="dr-library" deviceset="RESISTOR" device="0603" value="330"/>
+<part name="R1" library="dr-library" deviceset="RESISTOR" device="0805" value="10k"/>
+<part name="R2" library="dr-library" deviceset="RESISTOR" device="0805" value="330"/>
 <part name="S1" library="dr-library" deviceset="SKHMQME010" device=""/>
 <part name="C9" library="dr-library" deviceset="CAP" device="0603" value="1uF"/>
@@
 <part name="+3V6" library="supply1" deviceset="+3V3" device=""/>
 <part name="GND9" library="supply1" deviceset="GND" device=""/>
-<part name="R3" library="dr-library" deviceset="RESISTOR" device="0603" value="330"/>
+<part name="R3" library="dr-library" deviceset="RESISTOR" device="0805" value="330"/>
 <part name="D1" library="dr-library" deviceset="LED" device="1206" value="3V3"/>
 <part name="GND10" library="supply1" deviceset="GND" device=""/>
@@
 <part name="+3V9" library="supply1" deviceset="+3V3" device=""/>
 <part name="VREF_EN" library="dr-library" deviceset="M03" device=""/>
-<part name="R4" library="dr-library" deviceset="RESISTOR" device="0603" value="10k"/>
+<part name="R4" library="dr-library" deviceset="RESISTOR" device="0805" value="10k"/>
 <part name="+3V10" library="supply1" deviceset="+3V3" device=""/>
 <part name="GND13" library="supply1" deviceset="GND" device=""/>
@@
 <part name="GND14" library="supply1" deviceset="GND" device=""/>
 <part name="U$1" library="dr-library" deviceset="M03" device=""/>
-<part name="R5" library="dr-library" deviceset="RESISTOR" device="0603" value="330"/>
+<part name="R5" library="dr-library" deviceset="RESISTOR" device="0805" value="330"/>
 <part name="D2" library="dr-library" deviceset="LED" device="1206" value="PWR"/>
 <part name="GND15" library="supply1" deviceset="GND" device=""/>
@@
 <part name="GND20" library="supply1" deviceset="GND" device=""/>
 <part name="Q1" library="dr-library" deviceset="2N7002" device=""/>
-<part name="R6" library="dr-library" deviceset="RESISTOR" device="0603" value="330"/>
+<part name="R6" library="dr-library" deviceset="RESISTOR" device="0805" value="330"/>
 <part name="D3" library="dr-library" deviceset="LED" device="1206" value="PWR"/>
 <part name="+3V15" library="supply1" deviceset="+3V3" device=""/>
 <part name="GND21" library="supply1" deviceset="GND" device=""/>
 <part name="JP10" library="dr-library" deviceset="M02" device=""/>
-<part name="R7" library="dr-library" deviceset="RESISTOR" device="0603" value="10k"/>
+<part name="R7" library="dr-library" deviceset="RESISTOR" device="0805" value="10k"/>
 <part name="Q2" library="dr-library" deviceset="2N7002" device=""/>
-<part name="R8" library="dr-library" deviceset="RESISTOR" device="0603" value="330"/>
+<part name="R8" library="dr-library" deviceset="RESISTOR" device="0805" value="330"/>
 <part name="D4" library="dr-library" deviceset="LED" device="1206" value="PWR"/>
 <part name="+3V16" library="supply1" deviceset="+3V3" device=""/>
 <part name="GND22" library="supply1" deviceset="GND" device=""/>
 <part name="JP11" library="dr-library" deviceset="M02" device=""/>
-<part name="R9" library="dr-library" deviceset="RESISTOR" device="0603" value="10k"/>
+<part name="R9" library="dr-library" deviceset="RESISTOR" device="0805" value="10k"/>
 <part name="J2" library="EmbeddedAdventures 3" deviceset="JACK-PLUG" device="0"/>
 <part name="D5" library="dr-library" deviceset="VS-10BQ030-M3" device=""/>
@@
 <part name="GND1" library="supply1" deviceset="GND" device=""/>
 <part name="+3V14" library="supply1" deviceset="+3V3" device=""/>
-<part name="R10" library="dr-library" deviceset="RESISTOR" device="0603" value="10k"/>
+<part name="R10" library="dr-library" deviceset="RESISTOR" device="0805" value="10k"/>
 <part name="P+5" library="supply1" deviceset="VCC" device=""/>
 <part name="C17" library="dr-library" deviceset="CAP" device="0603" value="100nF"/>
 <part name="GND24" library="supply1" deviceset="GND" device=""/>
 <part name="USB_EN" library="dr-library" deviceset="M03" device=""/>
-<part name="R11" library="dr-library" deviceset="RESISTOR" device="0603" value="10k"/>
+<part name="R11" library="dr-library" deviceset="RESISTOR" device="0805" value="10k"/>
 <part name="GND25" library="supply1" deviceset="GND" device=""/>
 <part name="U5" library="dr-library" deviceset="AP7362-33SP-13" device=""/>
