File: ESP32 breakout/ESP32_breakout v2/ESP32_breakout v2.sch (EAGLE design)
At the start: 29 parts, among them U1 ESP-WROOM-32, U2 NCP-1117, Y1 12MHz

Commit message: Resized PCB v2
Parts:
- removed U$2: M04, dr-library:M04
Connections:
- net +3V3: no longer U$2.4
- net GND: no longer U$2.3
- net RX: no longer U$2.1
- net TX: no longer U$2.2
Changed lines of the file:
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@@
 <part name="U$17" library="dr-library" deviceset="M10" device="2X05"/>
 <part name="U$5" library="dr-library" deviceset="M10" device="2X05"/>
-<part name="U$2" library="dr-library" deviceset="M04" device=""/>
 <part name="U$3" library="dr-library" deviceset="M12" device="2ROWS"/>
 </parts>
@@
 <instance part="U$17" gate="G$1" x="83.82" y="2.54" rot="R180"/>
 <instance part="U$5" gate="G$1" x="177.8" y="2.54" rot="R180"/>
-<instance part="U$2" gate="G$1" x="177.8" y="-27.94" rot="R180"/>
 <instance part="U$3" gate="G$1" x="127" y="0" rot="R180"/>
 </instances>
@@
 </segment>
 <segment>
-<pinref part="U$2" gate="G$1" pin="3"/>
 <wire x1="172.72" y1="-30.48" x2="165.1" y2="-30.48" width="0.1524" layer="91"/>
 <label x="165.1" y="-30.48" size="1.778" layer="95"/>
@@
 </segment>
 <segment>
-<pinref part="U$2" gate="G$1" pin="4"/>
 <wire x1="172.72" y1="-27.94" x2="165.1" y2="-27.94" width="0.1524" layer="91"/>
 <label x="165.1" y="-27.94" size="1.778" layer="95"/>
@@
 </segment>
 <segment>
-<pinref part="U$2" gate="G$1" pin="2"/>
 <wire x1="172.72" y1="-33.02" x2="165.1" y2="-33.02" width="0.1524" layer="91"/>
 <label x="165.1" y="-33.02" size="1.778" layer="95"/>
@@
 </segment>
 <segment>
-<pinref part="U$2" gate="G$1" pin="1"/>
 <wire x1="172.72" y1="-35.56" x2="165.1" y2="-35.56" width="0.1524" layer="91"/>
 <label x="165.1" y="-35.56" size="1.778" layer="95"/>

Commit message: Finished major traces
Parts:
- removed U$3: M122ROWS, dr-library:M122ROWS
- added U$10: M04, dr-library:M04
- added U$2: M102X05, dr-library:M102X05
Connections:
- net +3V3: now also U$10.4
- net GND: now also U$10.3
- net IO0: now also U$2.1; no longer U$3.1
- net IO16: now also U$2.3; no longer U$3.3
- net IO17: now also U$2.4; no longer U$3.4
- net IO18: now also U$2.6; no longer U$3.6
- net IO19: now also U$2.7; no longer U$3.7
- net IO21: now also U$2.8; no longer U$3.8
- net IO22: now also U$2.9; no longer U$3.11
- net IO23: now also U$2.10; no longer U$3.12
- net IO4: now also U$2.2; no longer U$3.2
- net IO5: now also U$2.5; no longer U$3.5
- net RX: now also U$10.1; no longer U$3.9
- net TX: now also U$10.2; no longer U$3.10
Changed lines of the file:
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@@
 <part name="U$17" library="dr-library" deviceset="M10" device="2X05"/>
 <part name="U$5" library="dr-library" deviceset="M10" device="2X05"/>
-<part name="U$3" library="dr-library" deviceset="M12" device="2ROWS"/>
+<part name="U$2" library="dr-library" deviceset="M10" device="2X05"/>
+<part name="U$10" library="dr-library" deviceset="M04" device=""/>
 </parts>
 <sheets>
@@
 <instance part="U$17" gate="G$1" x="83.82" y="2.54" rot="R180"/>
 <instance part="U$5" gate="G$1" x="177.8" y="2.54" rot="R180"/>
-<instance part="U$3" gate="G$1" x="127" y="0" rot="R180"/>
+<instance part="U$2" gate="G$1" x="205.74" y="-2.54" rot="R180"/>
+<instance part="U$10" gate="G$1" x="177.8" y="-27.94" rot="R180"/>
 </instances>
 <busses>
@@
 <wire x1="172.72" y1="-30.48" x2="165.1" y2="-30.48" width="0.1524" layer="91"/>
 <label x="165.1" y="-30.48" size="1.778" layer="95"/>
+<pinref part="U$10" gate="G$1" pin="3"/>
 </segment>
 </net>
@@
 <wire x1="172.72" y1="-27.94" x2="165.1" y2="-27.94" width="0.1524" layer="91"/>
 <label x="165.1" y="-27.94" size="1.778" layer="95"/>
+<pinref part="U$10" gate="G$1" pin="4"/>
 </segment>
 </net>
@@
 <wire x1="121.92" y1="5.08" x2="114.3" y2="5.08" width="0.1524" layer="91"/>
 <label x="114.3" y="5.08" size="1.778" layer="95" font="vector"/>
-<pinref part="U$3" gate="G$1" pin="10"/>
 </segment>
 <segment>
@@
 <label x="165.1" y="-33.02" size="1.778" layer="95"/>
 <label x="165.1" y="-33.02" size="1.778" layer="95"/>
+<pinref part="U$10" gate="G$1" pin="2"/>
 </segment>
 </net>
@@
 <wire x1="121.92" y1="2.54" x2="114.3" y2="2.54" width="0.1524" layer="91"/>
 <label x="114.3" y="2.54" size="1.778" layer="95" font="vector"/>
-<pinref part="U$3" gate="G$1" pin="9"/>
 </segment>
 <segment>
@@
 <wire x1="172.72" y1="-35.56" x2="165.1" y2="-35.56" width="0.1524" layer="91"/>
 <label x="165.1" y="-35.56" size="1.778" layer="95"/>
+<pinref part="U$10" gate="G$1" pin="1"/>
 </segment>
 </net>
@@
 <wire x1="121.92" y1="-15.24" x2="114.3" y2="-15.24" width="0.1524" layer="91"/>
 <label x="114.3" y="-15.24" size="1.778" layer="95" font="vector"/>
-<pinref part="U$3" gate="G$1" pin="2"/>
+</segment>
+<segment>
+<wire x1="200.66" y1="-17.78" x2="193.04" y2="-17.78" width="0.1524" layer="91"/>
+<label x="193.04" y="-17.78" size="1.778" layer="95" font="vector"/>
+<pinref part="U$2" gate="G$1" pin="2"/>
 </segment>
 </net>
@@
 <wire x1="121.92" y1="-7.62" x2="114.3" y2="-7.62" width="0.1524" layer="91"/>
 <label x="114.3" y="-7.62" size="1.778" layer="95" font="vector"/>
-<pinref part="U$3" gate="G$1" pin="5"/>
+</segment>
+<segment>
+<wire x1="200.66" y1="-10.16" x2="193.04" y2="-10.16" width="0.1524" layer="91"/>
+<label x="193.04" y="-10.16" size="1.778" layer="95" font="vector"/>
+<pinref part="U$2" gate="G$1" pin="5"/>
 </segment>
 </net>
@@
 <wire x1="121.92" y1="-5.08" x2="114.3" y2="-5.08" width="0.1524" layer="91"/>
 <label x="114.3" y="-5.08" size="1.778" layer="95" font="vector"/>
-<pinref part="U$3" gate="G$1" pin="6"/>
+</segment>
+<segment>
+<wire x1="200.66" y1="-7.62" x2="193.04" y2="-7.62" width="0.1524" layer="91"/>
+<label x="193.04" y="-7.62" size="1.778" layer="95" font="vector"/>
+<pinref part="U$2" gate="G$1" pin="6"/>
 </segment>
 </net>
@@
 <wire x1="121.92" y1="-2.54" x2="114.3" y2="-2.54" width="0.1524" layer="91"/>
 <label x="114.3" y="-2.54" size="1.778" layer="95" font="vector"/>
-<pinref part="U$3" gate="G$1" pin="7"/>
+</segment>
+<segment>
+<wire x1="200.66" y1="-5.08" x2="193.04" y2="-5.08" width="0.1524" layer="91"/>
+<label x="193.04" y="-5.08" size="1.778" layer="95" font="vector"/>
+<pinref part="U$2" gate="G$1" pin="7"/>
 </segment>
 </net>
@@
 <wire x1="121.92" y1="0" x2="114.3" y2="0" width="0.1524" layer="91"/>
 <label x="114.3" y="0" size="1.778" layer="95" font="vector"/>
-<pinref part="U$3" gate="G$1" pin="8"/>
+</segment>
+<segment>
+<wire x1="200.66" y1="-2.54" x2="193.04" y2="-2.54" width="0.1524" layer="91"/>
+<label x="193.04" y="-2.54" size="1.778" layer="95" font="vector"/>
+<pinref part="U$2" gate="G$1" pin="8"/>
 </segment>
 </net>
@@
 <wire x1="121.92" y1="7.62" x2="114.3" y2="7.62" width="0.1524" layer="91"/>
 <label x="114.3" y="7.62" size="1.778" layer="95" font="vector"/>
-<pinref part="U$3" gate="G$1" pin="11"/>
+</segment>
+<segment>
+<wire x1="200.66" y1="0" x2="193.04" y2="0" width="0.1524" layer="91"/>
+<label x="193.04" y="0" size="1.778" layer="95" font="vector"/>
+<pinref part="U$2" gate="G$1" pin="9"/>
 </segment>
 </net>
@@
 <wire x1="121.92" y1="10.16" x2="114.3" y2="10.16" width="0.1524" layer="91"/>
 <label x="114.3" y="10.16" size="1.778" layer="95" font="vector"/>
-<pinref part="U$3" gate="G$1" pin="12"/>
+</segment>
+<segment>
+<wire x1="200.66" y1="2.54" x2="193.04" y2="2.54" width="0.1524" layer="91"/>
+<label x="193.04" y="2.54" size="1.778" layer="95" font="vector"/>
+<pinref part="U$2" gate="G$1" pin="10"/>
 </segment>
 </net>
@@
 <wire x1="121.92" y1="-10.16" x2="114.3" y2="-10.16" width="0.1524" layer="91"/>
 <label x="114.3" y="-10.16" size="1.778" layer="95" font="vector"/>
-<pinref part="U$3" gate="G$1" pin="4"/>
+</segment>
+<segment>
+<wire x1="200.66" y1="-12.7" x2="193.04" y2="-12.7" width="0.1524" layer="91"/>
+<label x="193.04" y="-12.7" size="1.778" layer="95" font="vector"/>
+<pinref part="U$2" gate="G$1" pin="4"/>
 </segment>
 </net>
@@
 <wire x1="121.92" y1="-12.7" x2="114.3" y2="-12.7" width="0.1524" layer="91"/>
 <label x="114.3" y="-12.7" size="1.778" layer="95" font="vector"/>
-<pinref part="U$3" gate="G$1" pin="3"/>
+</segment>
+<segment>
+<wire x1="200.66" y1="-15.24" x2="193.04" y2="-15.24" width="0.1524" layer="91"/>
+<label x="193.04" y="-15.24" size="1.778" layer="95" font="vector"/>
+<pinref part="U$2" gate="G$1" pin="3"/>
 </segment>
 </net>
@@
 <wire x1="121.92" y1="-17.78" x2="114.3" y2="-17.78" width="0.1524" layer="91"/>
 <label x="114.3" y="-17.78" size="1.778" layer="95" font="vector"/>
-<pinref part="U$3" gate="G$1" pin="1"/>
-</segment>
-</net>
+</segment>
+<segment>
+<wire x1="200.66" y1="-20.32" x2="193.04" y2="-20.32" width="0.1524" layer="91"/>
+<label x="193.04" y="-20.32" size="1.778" layer="95" font="vector"/>
+<pinref part="U$2" gate="G$1" pin="1"/>
+</segment>
+</net>

Commit message: Version 2, pre-check
Parts:
- renumbered U$16 to D2
Changed lines of the file:
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@@
 <part name="GND14" library="supply1" deviceset="GND" device=""/>
 <part name="J1" library="EmbeddedAdventures 3" deviceset="JACK-PLUG" device="0"/>
-<part name="U$16" library="EmbeddedAdventures 3" deviceset="DIODE-10BQ015PBF" device=""/>
+<part name="D2" library="EmbeddedAdventures 3" deviceset="DIODE-10BQ015PBF" device=""/>
 <part name="P+5" library="supply1" deviceset="VCC" device=""/>
 <part name="GND15" library="supply1" deviceset="GND" device=""/>
@@
 <instance part="GND14" gate="1" x="139.7" y="-20.32"/>
 <instance part="J1" gate="G$1" x="-5.08" y="114.3"/>
-<instance part="U$16" gate="G$1" x="7.62" y="116.84"/>
+<instance part="D2" gate="G$1" x="7.62" y="116.84"/>
 <instance part="P+5" gate="VCC" x="17.78" y="124.46"/>
 <instance part="GND15" gate="1" x="17.78" y="91.44"/>
@@
 </segment>
 <segment>
-<pinref part="U$16" gate="G$1" pin="C"/>
+<pinref part="D2" gate="G$1" pin="C"/>
 <wire x1="10.16" y1="116.84" x2="17.78" y2="116.84" width="0.1524" layer="91"/>
 <wire x1="17.78" y1="116.84" x2="17.78" y2="121.92" width="0.1524" layer="91"/>
@@
 <segment>
 <pinref part="J1" gate="G$1" pin="3"/>
-<pinref part="U$16" gate="G$1" pin="A"/>
+<pinref part="D2" gate="G$1" pin="A"/>
 <wire x1="0" y1="116.84" x2="5.08" y2="116.84" width="0.1524" layer="91"/>
 </segment>
@@
 </sheet>
 </sheets>
+<errors>
+</errors>
 </schematic>
 </drawing>
