File: Verification/verify.brd (EAGLE design)
At the start: 100 x 80 mm, 12 parts

Commit message: Edited packages
Parts:
- removed U$1: CAPACITOR0402, DR_passives:CAP-0402
- removed U$4: RESISTORR0402, DR_passives:RES-0402
- removed U$5: RESISTORR0603, DR_passives:RES-0603
- removed U$6: RESISTORR0805, DR_passives:RES-0805
- added C6: (no value), DR_passives:CAP-0402
- added R4: (no value), DR_passives:RES-0402
- added R5: (no value), DR_passives:RES-0603
- added R6: (no value), DR_passives:RES-0805
- C7: value CAPACITOR0603 -> (none)
- C8: value CAPACITOR0805 -> (none)
- moved R1 1.27 mm to (3.81, 12.7)
- moved R2 1.27 mm to (12.7, 12.7)
- moved R3 1.27 mm to (22.9, 12.7)
- renumbered U$2 to C7, U$3 to C8
Changed lines of the file:
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@@
 <element name="C2" library="EmbeddedAdventures 3" package="0603-CAP" value="" x="12.7" y="20.32"/>
 <element name="C3" library="EmbeddedAdventures 3" package="0805" value="" x="22.86" y="20.32"/>
-<element name="U$1" library="DR_passives" package="CAP-0402" value="CAPACITOR0402" x="3.81" y="19.05"/>
-<element name="U$2" library="DR_passives" package="CAP-0603" value="CAPACITOR0603" x="12.7" y="17.78"/>
-<element name="U$3" library="DR_passives" package="CAP-0805" value="CAPACITOR0805" x="22.86" y="17.78"/>
-<element name="R1" library="EmbeddedAdventures 3" package="0402-RES" value="" x="3.81" y="13.97"/>
-<element name="R2" library="EmbeddedAdventures 3" package="0603-RES" value="" x="12.7" y="13.97"/>
-<element name="R3" library="EmbeddedAdventures 3" package="0805" value="" x="22.86" y="13.97"/>
-<element name="U$4" library="DR_passives" package="RES-0402" value="RESISTORR0402" x="3.81" y="11.43"/>
-<element name="U$5" library="DR_passives" package="RES-0603" value="RESISTORR0603" x="12.7" y="11.43"/>
-<element name="U$6" library="DR_passives" package="RES-0805" value="RESISTORR0805" x="22.86" y="11.43"/>
+<element name="R1" library="EmbeddedAdventures 3" package="0402-RES" value="" x="3.81" y="12.7"/>
+<element name="R2" library="EmbeddedAdventures 3" package="0603-RES" value="" x="12.7" y="12.7"/>
+<element name="R3" library="EmbeddedAdventures 3" package="0805" value="" x="22.86" y="12.7"/>
+<element name="R4" library="DR_passives" package="RES-0402" value="" x="3.81" y="10.16"/>
+<element name="R5" library="DR_passives" package="RES-0603" value="" x="12.7" y="10.16"/>
+<element name="R6" library="DR_passives" package="RES-0805" value="" x="22.86" y="10.16"/>
+<element name="C6" library="DR_passives" package="CAP-0402" value="" x="3.81" y="17.78"/>
+<element name="C7" library="DR_passives" package="CAP-0603" value="" x="12.7" y="17.78"/>
+<element name="C8" library="DR_passives" package="CAP-0805" value="" x="22.86" y="17.78"/>
 </elements>
 <signals>

Commit message: Printout of Xbee
Parts:
- added U1: XBEE_S2C_SMDSMD, dr-library:XBEE_S2C_SMD
Changed lines of the file:
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@@
 <element name="C7" library="DR_passives" package="CAP-0603" value="" x="12.7" y="17.78"/>
 <element name="C8" library="DR_passives" package="CAP-0805" value="" x="22.86" y="17.78"/>
+<element name="U1" library="dr-library" package="XBEE_S2C_SMD" value="XBEE_S2C_SMDSMD" x="43.18" y="21.59"/>
 </elements>
 <signals>
