File: Verification/verify.sch (EAGLE design)
At the start: 12 parts

Commit message: Edited packages
Parts:
- removed U$1: CAPACITOR0402, DR_passives:CAPACITOR0402
- removed U$2: CAPACITOR0603, DR_passives:CAPACITOR0603
- removed U$3: CAPACITOR0805, DR_passives:CAPACITOR0805
- removed U$4: RESISTORR0402, DR_passives:RESISTORR0402
- removed U$5: RESISTORR0603, DR_passives:RESISTORR0603
- removed U$6: RESISTORR0805, DR_passives:RESISTORR0805
- added C6: (no value), DR_passives:CAPACITOR0402
- added C7: (no value), DR_passives:CAPACITOR0603
- added C8: (no value), DR_passives:CAPACITOR0805
- added R4: (no value), DR_passives:RESISTOR0402
- added R5: (no value), DR_passives:RESISTOR0603
- added R6: (no value), DR_passives:RESISTOR0805
Changed lines of the file:
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@@
 <part name="C2" library="EmbeddedAdventures 3" deviceset="CAP" device="0603-CAP"/>
 <part name="C3" library="EmbeddedAdventures 3" deviceset="CAP" device="0805"/>
-<part name="U$1" library="DR_passives" deviceset="CAPACITOR" device="0402"/>
-<part name="U$2" library="DR_passives" deviceset="CAPACITOR" device="0603"/>
-<part name="U$3" library="DR_passives" deviceset="CAPACITOR" device="0805"/>
 <part name="R1" library="EmbeddedAdventures 3" deviceset="RESISTOR" device="0402-RES"/>
 <part name="R2" library="EmbeddedAdventures 3" deviceset="RESISTOR" device="0603-RES"/>
 <part name="R3" library="EmbeddedAdventures 3" deviceset="RESISTOR" device=""/>
-<part name="U$4" library="DR_passives" deviceset="RESISTOR" device="R0402"/>
-<part name="U$5" library="DR_passives" deviceset="RESISTOR" device="R0603"/>
-<part name="U$6" library="DR_passives" deviceset="RESISTOR" device="R0805"/>
+<part name="R4" library="DR_passives" deviceset="RESISTOR" device="0402"/>
+<part name="R5" library="DR_passives" deviceset="RESISTOR" device="0603"/>
+<part name="R6" library="DR_passives" deviceset="RESISTOR" device="0805"/>
+<part name="C6" library="DR_passives" deviceset="CAPACITOR" device="0402"/>
+<part name="C7" library="DR_passives" deviceset="CAPACITOR" device="0603"/>
+<part name="C8" library="DR_passives" deviceset="CAPACITOR" device="0805"/>
 </parts>
 <sheets>
@@
 <instance part="C2" gate="G$1" x="7.62" y="15.24"/>
 <instance part="C3" gate="G$1" x="15.24" y="15.24"/>
-<instance part="U$1" gate="G$1" x="0" y="0"/>
-<instance part="U$2" gate="G$1" x="17.78" y="0"/>
-<instance part="U$3" gate="G$1" x="35.56" y="0"/>
 <instance part="R1" gate="G$1" x="-2.54" y="-17.78"/>
 <instance part="R2" gate="G$1" x="15.24" y="-17.78"/>
 <instance part="R3" gate="G$1" x="33.02" y="-17.78"/>
-<instance part="U$4" gate="G$1" x="-2.54" y="-30.48"/>
-<instance part="U$5" gate="G$1" x="20.32" y="-30.48"/>
-<instance part="U$6" gate="G$1" x="43.18" y="-30.48"/>
+<instance part="R4" gate="G$1" x="-2.54" y="-25.4"/>
+<instance part="R5" gate="G$1" x="15.24" y="-25.4"/>
+<instance part="R6" gate="G$1" x="33.02" y="-25.4"/>
+<instance part="C6" gate="G$1" x="0" y="-2.54"/>
+<instance part="C7" gate="G$1" x="7.62" y="-2.54"/>
+<instance part="C8" gate="G$1" x="15.24" y="-2.54"/>
 </instances>
 <busses>

Commit message: Printout of Xbee
Parts:
- added U1: XBEE_S2C_SMDSMD, dr-library:XBEE_S2C_SMDSMD
Changed lines of the file:
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@@
 <part name="C7" library="DR_passives" deviceset="CAPACITOR" device="0603"/>
 <part name="C8" library="DR_passives" deviceset="CAPACITOR" device="0805"/>
+<part name="U1" library="dr-library" deviceset="XBEE_S2C_SMD" device="SMD"/>
 </parts>
 <sheets>
@@
 <instance part="C7" gate="G$1" x="7.62" y="-2.54"/>
 <instance part="C8" gate="G$1" x="15.24" y="-2.54"/>
+<instance part="U1" gate="G$1" x="81.28" y="15.24"/>
 </instances>
 <busses>
